File: Hardware/Shuffleboard/_autosave-Shuffleboard.kicad_pcb (KiCad board)
At the start: 4 copper layers, 131 x 132.4 mm, 31 parts, among them J1 1751138, J2 1751138, U1 COM-09032, U2 PAM8302AAS

Commit message: led's, mux
Parts:
- J1, J2: value 1751138 -> 1869279; footprint ShuffleboardFootprints:1751138 -> ShuffleboardFootprints:1869279
- moved J1 117.0 mm to (232.5, 39.8)
- moved C6 80.3 mm to (96.5, 136.7)
- moved F1 80.3 mm to (96.5, 139.2)
- moved TP2 80.3 mm to (100.5, 134.8)
- moved C2 80.3 mm to (96.5, 134.2)
- moved U2 3.31 mm to (196.2, 107.5)
- moved J2 0.79 mm to (117.8, 38.5)
Connections:
- J1 pad 1: /DACOut -> /3.3VIN
- J1 pad 2: /PB4SHOOT -> /DACOut
- J1 pad 3: /PB1RST -> /PB4SHOOT
- J1 pad 4: /Connector/POS_PB17_ADC1_4 -> /PB1RST
- J1 pad 5: /Connector/HOR_PB18_ADC1_5 -> /Connector/POS_PB17_ADC1_4
- J1 pad 6: /Connector/VER_PB19_ADC1_6 -> /Connector/HOR_PB18_ADC1_5
- J2 pad 1: /3.3VIN -> unconnected-(J2-Pad1)
- J2 pad 6: /Connector/GNDIN -> unconnected-(J2-Pad6)
Routing:
- net /3.3VIN: track 0.00 -> 4.97 mm, vias 0 -> 1
- net /Connector/GNDIN: track 0.00 -> 4.55 mm, vias 0 -> 1
