File: Hardware/Shuffleboard/power.kicad_sch (KiCad schematic)
At the start: 4 parts

Commit message: led's, mux
Parts:
- added D32: Green, LED_THT:LED_D5.0mm, symbol Device:LED
- added R8: 1k, Resistor_SMD:R_0603_1608Metric_Pad0.98x0.95mm_HandSolder, symbol Device:R
Connections:
- net GND: now also D32.1 (K)
- new net: D32.2 (A), R8.1
- new net +3V3: R8.2
Other:
- note added: "Power Indicator"

Commit message: fet led driving
Connections:
- net +3V3 is gone; now on net +3.3V: R8.2
- net +3.3V: now also C2.1, C6.2, F1.2, TP2.1
Changed lines of the file:
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@@
+	)
+	(junction
+		(at 59.69 30.48)
+		(diameter 0)
+		(color 0 0 0 0)
 	)
 	(junction
@@
 	(symbol
 		(lib_id "power:+3.3V")
-		(at 60.96 30.48 0)
+		(at 59.69 30.48 0)
 		(unit 1)
 		(exclude_from_sim no)
@@
 		(fields_autoplaced yes)
 		(property "Reference" "#PWR025"
-			(at 60.96 34.29 0)
+			(at 59.69 34.29 0)
 			(effects
 				(font
@@
 		)
 		(property "Value" "+3.3V"
-			(at 60.96 25.4 0)
+			(at 59.69 25.4 0)
 			(effects
 				(font
@@
 		)
 		(property "Footprint" ""
-			(at 60.96 30.48 0)
+			(at 59.69 30.48 0)
 			(effects
 				(font
@@
 		)
 		(property "Datasheet" ""
-			(at 60.96 30.48 0)
+			(at 59.69 30.48 0)
 			(effects
 				(font
@@
 		)
 		(property "Description" "Power symbol creates a global label with name \"+3.3V\""
-			(at 60.96 30.48 0)
+			(at 59.69 30.48 0)
 			(effects
 				(font
@@
 			)
 		)
-		(property "Value" "+3V3"
+		(property "Value" "+3.3V"
 			(at 87.63 16.51 0)
 			(effects

Commit message: layout 2
Parts:
- added TP1: GND, TestPoint:TestPoint_THTPad_1.5x1.5mm_Drill0.7mm, symbol Connector:TestPoint
Connections:
- net GND: now also TP1.1
Changed lines of the file:
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@@
+		(color 0 0 0 0)
+	)
+	(junction
+		(at 45.72 38.1)
+		(diameter 0)
 		(color 0 0 0 0)
 	)
@@
 					(unit 1)
 				)
+			)
+		)
+	)
+	(symbol
+		(lib_id "Connector:TestPoint")
+		(at 45.72 38.1 90)
+		(unit 1)
+		(exclude_from_sim no)
+		(in_bom no)
+		(on_board yes)
+		(dnp no)
+		(property "Reference" "TP1"
+			(at 39.624 38.1 90)
+			(effects
+				(font
+					(size 1.27 1.27)
+				)
+			)
+		)
+		(property "Value" "GND"
+			(at 40.64 36.8301 90)
+			(effects
+				(font
+					(size 1.27 1.27)
+				)
+				(justify left)
+				(hide yes)
+			)
+		)
+		(property "Footprint" "TestPoint:TestPoint_THTPad_1.5x1.5mm_Drill0.7mm"
+			(at 45.72 33.02 0)
+			(effects
+				(font
+					(size 1.27 1.27)
+				)
+				(hide yes)
+			)
+		)
+		(property "Datasheet" "~"
+			(at 45.72 33.02 0)
+			(effects
+				(font
+					(size 1.27 1.27)
+				)
+				(hide yes)
+			)
+		)
+		(property "Description" "test point"
+			(at 45.72 38.1 0)
+			(effects
+				(font
+					(size 1.27 1.27)
+				)
+				(hide yes)
+			)
+		)
+		(property "Mouser Link" ""
+			(at 45.72 38.1 0)
+			(effects
+				(font
+					(size 1.27 1.27)
+				)
+				(hide yes)
+			)
+		)
+		(property "JLCPCB #" ""
+			(at 45.72 38.1 0)
+			(effects
+				(font
+					(size 1.27 1.27)
+				)
+				(hide yes)
+			)
+		)
+		(pin "1"
+		)
+		(instances
+			(project "Shuffleboard"
+				(path "/8d05e546-da1a-40d0-9e47-08c4b800bb0e/52b4f5df-1b13-4b39-b0ff-c702f38956fb"
+					(reference "TP1")
+					(unit 1)
+				)

Commit message: finished layout
Parts:
- C2: value 4.7u -> (none)
- C6: value 100n -> (none)
- D32: value Green -> (none)
- F1: value 1A -> (none)
- R8: value 1k -> (none); footprint Resistor_SMD:R_0603_1608Metric_Pad0.98x0.95mm_HandSolder -> Resistor_THT:R_Axial_DIN0207_L6.3mm_D2.5mm_P7.62mm_Horizontal
- TP1: value GND -> (none)
- TP2: value +3.3 -> (none)

Commit message: tht resistors
Parts:
- C2, C6: value (none) -> 100n
- D32: value (none) -> Green
- R8: value (none) -> 1k; now left out of the parts list
Changed lines of the file:
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@@
+			)
+		)
+		(property "VALUE" ""
+			(at 39.37 30.48 90)
+			(hide yes)
+			(show_name no)
+			(do_not_autoplace no)
+			(effects
+				(font
+					(size 1.27 1.27)
+				)
 			)
 		)
@@
 			)
 		)
+		(property "VALUE" ""
+			(at 59.69 30.48 90)
+			(hide yes)
+			(show_name no)
+			(do_not_autoplace no)
+			(effects
+				(font
+					(size 1.27 1.27)
+				)
+			)
+		)
 		(pin "1"
 		)
@@
 		(property "JLCPCB #" ""
 			(at 45.72 38.1 0)
+			(hide yes)
+			(show_name no)
+			(do_not_autoplace no)
+			(effects
+				(font
+					(size 1.27 1.27)
+				)
+			)
+		)
+		(property "VALUE" ""
+			(at 45.72 38.1 90)
 			(hide yes)
 			(show_name no)
@@
 		(body_style 1)
 		(exclude_from_sim no)
-		(in_bom yes)
+		(in_bom no)
 		(on_board yes)
 		(in_pos_files yes)
@@
 			)
 		)
-		(property "Value" ""
+		(property "Value" "1k"
 			(at 87.63 27.94 90)
 			(hide yes)
@@
 		)
 		(property "Mouser Part Number" "71-CRCW0603-1.0K-E3"
+			(at 87.63 27.94 90)
+			(hide yes)
+			(show_name no)
+			(do_not_autoplace no)
+			(effects
+				(font
+					(size 1.27 1.27)
+				)
+			)
+		)
+		(property "VALUE" ""
 			(at 87.63 27.94 90)
 			(hide yes)
@@
 			)
 		)
-		(property "Value" ""
+		(property "Value" "Green"
 			(at 87.63 35.56 90)
 			(hide yes)
@@
 		)
 		(property "Mouser Part Number" "710-151051VS04000"
+			(at 87.63 35.56 90)
+			(hide yes)
+			(show_name no)
+			(do_not_autoplace no)
+			(effects
+				(font
+					(size 1.27 1.27)
+				)
+			)
+		)
+		(property "VALUE" ""
 			(at 87.63 35.56 90)
 			(hide yes)
@@
 			)
 		)
-		(property "Value" ""
+		(property "Value" "100n"
 			(at 45.72 34.29 0)
 			(hide yes)
@@
 		)
 		(property "Mouser Part Number" "81-GRM188R6YA475KE5D"
+			(at 45.72 34.29 0)
+			(hide yes)
+			(show_name no)
+			(do_not_autoplace no)
+			(effects
+				(font
+					(size 1.27 1.27)
+				)
+			)
+		)
+		(property "VALUE" ""
 			(at 45.72 34.29 0)
 			(hide yes)
@@
 			)
 		)
-		(property "Value" ""
+		(property "Value" "100n"
 			(at 49.53 26.67 0)
 			(hide yes)
@@
 			(at 49.53 26.67 0)
 			(hide yes)
+			(show_name no)
+			(do_not_autoplace no)
+			(effects
+				(font
+					(size 1.27 1.27)
+				)
+			)
+		)
+		(property "VALUE" ""
+			(at 49.53 26.67 0)
+			(hide yes)

Commit message: updated to end
Parts:
- C2, C6: value 100n -> (none)
- D32: value Green -> (none)
- R8: value 1k -> (none)
Changed lines of the file:
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@@
-			)
-		)
-		(property "VALUE" ""
-			(at 39.37 30.48 90)
-			(hide yes)
-			(show_name no)
-			(do_not_autoplace no)
-			(effects
-				(font
-					(size 1.27 1.27)
-				)
 			)
 		)
@@
 			)
 		)
-		(property "VALUE" ""
-			(at 59.69 30.48 90)
-			(hide yes)
-			(show_name no)
-			(do_not_autoplace no)
-			(effects
-				(font
-					(size 1.27 1.27)
-				)
-			)
-		)
 		(pin "1"
 		)
@@
 		(property "JLCPCB #" ""
 			(at 45.72 38.1 0)
-			(hide yes)
-			(show_name no)
-			(do_not_autoplace no)
-			(effects
-				(font
-					(size 1.27 1.27)
-				)
-			)
-		)
-		(property "VALUE" ""
-			(at 45.72 38.1 90)
 			(hide yes)
 			(show_name no)
@@
 			)
 		)
-		(property "Value" "1k"
+		(property "Value" ""
 			(at 87.63 27.94 90)
 			(hide yes)
@@
 		)
 		(property "Mouser Part Number" "71-CRCW0603-1.0K-E3"
-			(at 87.63 27.94 90)
-			(hide yes)
-			(show_name no)
-			(do_not_autoplace no)
-			(effects
-				(font
-					(size 1.27 1.27)
-				)
-			)
-		)
-		(property "VALUE" ""
 			(at 87.63 27.94 90)
 			(hide yes)
@@
 			)
 		)
-		(property "Value" "Green"
+		(property "Value" ""
 			(at 87.63 35.56 90)
 			(hide yes)
@@
 		)
 		(property "Mouser Part Number" "710-151051VS04000"
-			(at 87.63 35.56 90)
-			(hide yes)
-			(show_name no)
-			(do_not_autoplace no)
-			(effects
-				(font
-					(size 1.27 1.27)
-				)
-			)
-		)
-		(property "VALUE" ""
 			(at 87.63 35.56 90)
 			(hide yes)
@@
 			)
 		)
-		(property "Value" "100n"
+		(property "Value" ""
 			(at 45.72 34.29 0)
 			(hide yes)
@@
 		)
 		(property "Mouser Part Number" "81-GRM188R6YA475KE5D"
-			(at 45.72 34.29 0)
-			(hide yes)
-			(show_name no)
-			(do_not_autoplace no)
-			(effects
-				(font
-					(size 1.27 1.27)
-				)
-			)
-		)
-		(property "VALUE" ""
 			(at 45.72 34.29 0)
 			(hide yes)
@@
 			)
 		)
-		(property "Value" "100n"
+		(property "Value" ""
 			(at 49.53 26.67 0)
 			(hide yes)
@@
 			(at 49.53 26.67 0)
 			(hide yes)
-			(show_name no)
-			(do_not_autoplace no)
-			(effects
-				(font
-					(size 1.27 1.27)
-				)
-			)
-		)
-		(property "VALUE" ""
-			(at 49.53 26.67 0)
-			(hide yes)
