File: Hardware/Shuffleboard/speaker.kicad_sch (KiCad schematic)
At the start: 5 parts, among them U2 PAM8302AAS

Commit message: fet led driving
Connections:
- net OUT-: now reaches LS1.N, U2.8 (OUT-)
- net OUT+: now reaches LS1.P, U2.5 (OUT+)
Changed lines of the file:
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@@
+		)
+	)
+	(label "OUT-"
+		(at 100.33 34.29 0)
+		(effects
+			(font
+				(size 1.27 1.27)
+			)
+			(justify left bottom)
+		)
+	)
+	(label "OUT+"
+		(at 100.33 24.13 0)
+		(effects
+			(font
+				(size 1.27 1.27)
+			)
+			(justify left bottom)
 		)
 	)

Commit message: finished layout
Parts:
- C8: value 100n -> (none)
- C9: value 1u -> (none)
- LS1: value CMS-3012-18T -> (none)
- R7: value 1k -> (none); footprint Resistor_SMD:R_0603_1608Metric_Pad0.98x0.95mm_HandSolder -> Resistor_THT:R_Axial_DIN0207_L6.3mm_D2.5mm_P7.62mm_Horizontal
- U2: value PAM8302AAS -> (none)

Commit message: finalized
Parts:
- added C12: 100n, Capacitor_SMD:C_0603_1608Metric_Pad1.08x0.95mm_HandSolder, symbol Device:C
Connections:
- net +3.3V: now also C12.1
- net GND: now also C12.2
Other:
- moved on the sheet: C8, C9, LS1, R7, U2

Commit message: tht resistors
Parts:
- C8: value (none) -> 100n
- C9: value (none) -> 1u
- R7: value (none) -> 1k; now left out of the parts list
Changed lines of the file:
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@@
+			)
+		)
+		(property "VALUE" ""
+			(at 80.01 25.4 0)
+			(hide yes)
+			(show_name no)
+			(do_not_autoplace no)
+			(effects
+				(font
+					(size 1.27 1.27)
+				)
 			)
 		)
@@
 			)
 		)
+		(property "VALUE" ""
+			(at 102.87 36.83 0)
+			(hide yes)
+			(show_name no)
+			(do_not_autoplace no)
+			(effects
+				(font
+					(size 1.27 1.27)
+				)
+			)
+		)
 		(pin "P"
 		)
@@
 		(body_style 1)
 		(exclude_from_sim no)
-		(in_bom yes)
+		(in_bom no)
 		(on_board yes)
 		(in_pos_files yes)
@@
 			)
 		)
-		(property "Value" ""
+		(property "Value" "1k"
 			(at 40.64 34.29 90)
 			(hide yes)
@@
 		)
 		(property "Mouser Part Number" "71-CRCW0603-1.0K-E3"
+			(at 40.64 34.29 90)
+			(hide yes)
+			(show_name no)
+			(do_not_autoplace no)
+			(effects
+				(font
+					(size 1.27 1.27)
+				)
+			)
+		)
+		(property "VALUE" ""
 			(at 40.64 34.29 90)
 			(hide yes)
@@
 		)
 		(property "Mouser Part Number" "621-PAM8302AASCR"
+			(at 76.2 39.37 0)
+			(hide yes)
+			(show_name no)
+			(do_not_autoplace no)
+			(effects
+				(font
+					(size 1.27 1.27)
+				)
+			)
+		)
+		(property "VALUE" ""
 			(at 76.2 39.37 0)
 			(hide yes)
@@
 			)
 		)
-		(property "Value" ""
+		(property "Value" "100n"
 			(at 44.45 38.1 0)
 			(hide yes)
@@
 		)
 		(property "Mouser Part Number" "581-06031C104K4T2A"
+			(at 44.45 38.1 0)
+			(hide yes)
+			(show_name no)
+			(do_not_autoplace no)
+			(effects
+				(font
+					(size 1.27 1.27)
+				)
+			)
+		)
+		(property "VALUE" ""
 			(at 44.45 38.1 0)
 			(hide yes)
@@
 			)
 		)
-		(property "Value" ""
+		(property "Value" "1u"
 			(at 57.15 34.29 90)
 			(hide yes)
@@
 			(at 57.15 34.29 90)
 			(hide yes)
+			(show_name no)
+			(do_not_autoplace no)
+			(effects
+				(font
+					(size 1.27 1.27)
+				)
+			)
+		)
+		(property "VALUE" ""
+			(at 57.15 34.29 90)
+			(hide yes)

Commit message: updated to end
Parts:
- C12, C8: value 100n -> (none)
- C9: value 1u -> (none)
- R7: value 1k -> (none)
Changed lines of the file:
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@@
 			)
 		)
-		(property "Value" "100n"
-			(at 81.026 19.304 0)
+		(property "Value" ""
+			(at 80.01 25.4 0)
+			(hide yes)
 			(show_name no)
 			(do_not_autoplace no)
@@
 		)
 		(property "Mouser Part Number" "581-06031C104K4T2A"
-			(at 80.01 25.4 0)
-			(hide yes)
-			(show_name no)
-			(do_not_autoplace no)
-			(effects
-				(font
-					(size 1.27 1.27)
-				)
-			)
-		)
-		(property "VALUE" ""
 			(at 80.01 25.4 0)
 			(hide yes)
@@
 			)
 		)
-		(property "VALUE" ""
-			(at 102.87 36.83 0)
-			(hide yes)
-			(show_name no)
-			(do_not_autoplace no)
-			(effects
-				(font
-					(size 1.27 1.27)
-				)
-			)
-		)
 		(pin "P"
 		)
@@
 			)
 		)
-		(property "Value" "1k"
+		(property "Value" ""
 			(at 40.64 34.29 90)
 			(hide yes)
@@
 		)
 		(property "Mouser Part Number" "71-CRCW0603-1.0K-E3"
-			(at 40.64 34.29 90)
-			(hide yes)
-			(show_name no)
-			(do_not_autoplace no)
-			(effects
-				(font
-					(size 1.27 1.27)
-				)
-			)
-		)
-		(property "VALUE" ""
 			(at 40.64 34.29 90)
 			(hide yes)
@@
 		)
 		(property "Mouser Part Number" "621-PAM8302AASCR"
-			(at 76.2 39.37 0)
-			(hide yes)
-			(show_name no)
-			(do_not_autoplace no)
-			(effects
-				(font
-					(size 1.27 1.27)
-				)
-			)
-		)
-		(property "VALUE" ""
 			(at 76.2 39.37 0)
 			(hide yes)
@@
 			)
 		)
-		(property "Value" "100n"
+		(property "Value" ""
 			(at 44.45 38.1 0)
 			(hide yes)
@@
 		)
 		(property "Mouser Part Number" "581-06031C104K4T2A"
-			(at 44.45 38.1 0)
-			(hide yes)
-			(show_name no)
-			(do_not_autoplace no)
-			(effects
-				(font
-					(size 1.27 1.27)
-				)
-			)
-		)
-		(property "VALUE" ""
 			(at 44.45 38.1 0)
 			(hide yes)
@@
 			)
 		)
-		(property "Value" "1u"
+		(property "Value" ""
 			(at 57.15 34.29 90)
 			(hide yes)
@@
 			(at 57.15 34.29 90)
 			(hide yes)
-			(show_name no)
-			(do_not_autoplace no)
-			(effects
-				(font
-					(size 1.27 1.27)
-				)
-			)
-		)
-		(property "VALUE" ""
-			(at 57.15 34.29 90)
-			(hide yes)
